Commit message: Add files via upload

File: romr_ros/src/urdf/romr_robot.xacro (robot description, xacro)
@@ -1,8 +1,8 @@
 <?xml version="1.0" encoding="utf-8"?>
-<robot name="romr_robot" xmlns:xacro="http://www.ros.org/wiki/xacro">
-<xacro:include filename="$(find romr_robot)/urdf/romr_materials.xacro" />
-<xacro:include filename="$(find romr_robot)/gazebo/romr_gazebo_materials.gazebo" />
-<xacro:include filename="$(find romr_robot)/gazebo/romr_gazebo_physics.gazebo" />
-<xacro:include filename="$(find romr_robot)/gazebo/romr_gazebo_plugins.gazebo" />
+<robot name="romr_ros" xmlns:xacro="http://www.ros.org/wiki/xacro">
+<xacro:include filename="$(find romr_ros)/urdf/romr_materials.xacro" />
+<xacro:include filename="$(find romr_ros)/gazebo/romr_gazebo_materials.gazebo" />
+<xacro:include filename="$(find romr_ros)/gazebo/romr_gazebo_physics.gazebo" />
+<xacro:include filename="$(find romr_ros)/gazebo/romr_gazebo_plugins.gazebo" />
   <!--******** Define intertial property macros ********** -->
   <xacro:macro name="footprint_inertia" params="m w h d">
@@ -33,5 +33,5 @@
       <origin xyz="0 0 0" rpy="0 0 0" />
       <geometry>
-        <mesh filename="package://romr_robot/meshes/base_link.STL" />
+        <mesh filename="package://romr_ros/meshes/base_link.STL" />
       </geometry>
       <material name="white">
@@ -41,5 +41,5 @@
       <origin xyz="0 0 0" rpy="0 0 0" />
       <geometry>
-        <mesh filename="package://romr_robot/meshes/base_link.STL" />
+        <mesh filename="package://romr_ros/meshes/base_link.STL" />
       </geometry>
     </collision>
@@ -54,5 +54,5 @@
       <origin xyz="0 0 0" rpy="0 0 0" />
       <geometry>
-        <mesh filename="package://romr_robot/meshes/rightwheel.STL" />
+        <mesh filename="package://romr_ros/meshes/rightwheel.STL" />
       </geometry>
       <material name="black">
@@ -62,5 +62,5 @@
       <origin xyz="0 0 0"  rpy="0 0 0" />
       <geometry>
-        <mesh filename="package://romr_robot/meshes/rightwheel.STL" />
+        <mesh filename="package://romr_ros/meshes/rightwheel.STL" />
       </geometry>
     </collision>
@@ -81,5 +81,5 @@
       <origin xyz="0 0 0" rpy="0 0 0" />
       <geometry>
-        <mesh filename="package://romr_robot/meshes/leftwheel.STL" />
+        <mesh filename="package://romr_ros/meshes/leftwheel.STL" />
       </geometry>
       <material name="black">
@@ -89,5 +89,5 @@
       <origin xyz="0 0 0" rpy="0 0 0" />
       <geometry>
-        <mesh filename="package://romr_robot/meshes/leftwheel.STL" />
+        <mesh filename="package://romr_ros/meshes/leftwheel.STL" />
       </geometry>
     </collision>
@@ -108,5 +108,5 @@
       <origin xyz="0 0 0" rpy="0 0 0" />
       <geometry>
-        <mesh filename="package://romr_robot/meshes/casterwheel.STL" />
+        <mesh filename="package://romr_ros/meshes/casterwheel.STL" />
       </geometry>
       <material name="blue">
@@ -116,5 +116,5 @@
       <origin xyz="0 0 0" rpy="0 0 0" />
       <geometry>
-        <mesh filename="package://romr_robot/meshes/casterwheel.STL" />
+        <mesh filename="package://romr_ros/meshes/casterwheel.STL" />
       </geometry>
     </collision>
@@ -135,5 +135,5 @@
       <origin xyz="0 0 0" rpy="0 0 0" />
       <geometry>
-        <mesh filename="package://romr_robot/meshes/lidar.STL" />
+        <mesh filename="package://romr_ros/meshes/lidar.STL" />
       </geometry>
       <material name="grey">
@@ -143,5 +143,5 @@
       <origin  xyz="0 0 0" rpy="0 0 0" />
       <geometry>
-        <mesh filename="package://romr_robot/meshes/lidar.STL" />
+        <mesh filename="package://romr_ros/meshes/lidar.STL" />
       </geometry>
     </collision>
@@ -162,5 +162,5 @@
       <origin xyz="0 0 0" rpy="0 0 0" />
       <geometry>
-        <mesh filename="package://romr_robot/meshes/imu.STL" />
+        <mesh filename="package://romr_ros/meshes/imu.STL" />
       </geometry>
       <material name="black">
@@ -170,5 +170,5 @@
       <origin xyz="0 0 0" rpy="0 0 0" />
       <geometry>
-        <mesh filename="package://romr_robot/meshes/imu.STL" />
+        <mesh filename="package://romr_ros/meshes/imu.STL" />
       </geometry>
     </collision>
@@ -189,5 +189,5 @@
       <origin xyz="0 0 0" rpy="0 0 0" />
       <geometry>
-        <mesh filename="package://romr_robot/meshes/camerad435i.STL" />
+        <mesh filename="package://romr_ros/meshes/camerad435i.STL" />
       </geometry>
       <material name="white">
@@ -197,5 +197,5 @@
       <origin xyz="0 0 0" rpy="0 0 0" />
       <geometry>
-        <mesh filename="package://romr_robot/meshes/camerad435i.STL" />
+        <mesh filename="package://romr_ros/meshes/camerad435i.STL" />
       </geometry>
     </collision>
@@ -216,5 +216,5 @@
       <origin  xyz="0 0 0"  rpy="0 0 0" />
       <geometry>
-        <mesh filename="package://romr_robot/meshes/camerat265.STL" />
+        <mesh filename="package://romr_ros/meshes/camerat265.STL" />
       </geometry>
       <material name="white">
@@ -224,5 +224,5 @@
       <origin xyz="0 0 0" rpy="0 0 0" />
       <geometry>
-        <mesh filename="package://romr_robot/meshes/camerat265.STL" />
+        <mesh filename="package://romr_ros/meshes/camerat265.STL" />
       </geometry>
     </collision>
